File: StickHub.kicad_pcb (KiCad board)
At the start: 2 copper layers, 16.5 x 40 mm, 94 parts, among them J1 HOST, J2 USB1, J3 USB2, J4 USB3, J5 USB4, J6 USB5, J7 USB6, J8 USB7, J9 EXTGND, U1 MaxLinear_XR22417-48, U2 Dialog_SLG5NT1487V, Y1 12MHz 50ppm 16-20pF

Commit message: Bump silkscreen version to v1.4.1
Other:
- board text added: "7-PORT USB 2.0 HUB v1.4.1 rbts.co/h1"
- board text removed: "7-PORT USB 2.0 HUB v1.4.0 rbts.co/h1"
Changed lines of the file:
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@@
 		)
 	)
-	(gr_text "7-PORT USB\n2.0 HUB v1.4.0\nrbts.co/h1"
+	(gr_text "7-PORT USB\n2.0 HUB v1.4.1\nrbts.co/h1"
 		(at 146.75 119.5 90)
 		(layer "B.SilkS")
